File: _autosave-tps61040DBVR-boost-converter-module.kicad_sch (KiCad schematic)
At the start: 12 parts, among them J1 +5V, J2 +12V, J3 GND, J4 GND, U1 TPS61040DBVR

Commit message: Media
Other:
- note added: "TPS61040DBVR 5V TO 12V BOOST CONVERTER"
Changed lines of the file:
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@@
+		)
+	)
+	(text "TPS61040DBVR 5V TO 12V BOOST CONVERTER"
+		(exclude_from_sim no)
+		(at 149.86 64.77 0)
+		(effects
+			(font
+				(size 4 4)
+				(thickness 0.4)
+				(bold yes)
+			)
 		)
 	)
