File: tps61040DBVR-boost-converter-module.kicad_pcb (KiCad board)
At the start: 2 copper layers, 18 x 13.5 mm, 12 parts, among them U1 TPS61040DBVR

Commit message: Media
Parts:
- moved 12V 0.50 mm to (196.6, 101.5)
- moved 5V 0.50 mm to (180.9, 101.5)
Other:
- board size 18 x 13.5 mm -> 18 x 14 mm
Changed lines of the file:
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@@
 	(footprint "Connector_PinHeader_1.00mm:PinHeader_1x01_P1.00mm_Vertical"
 		(layer "F.Cu")
-		(at 180.865 100.975)
+		(at 180.865 101.475)
 		(descr "Through hole straight pin header, 1x01, 1.00mm pitch, single row")
 		(tags "Through hole pin header THT 1x01 1.00mm single row")
@@
 	(footprint "Connector_PinHeader_1.00mm:PinHeader_1x01_P1.00mm_Vertical"
 		(layer "F.Cu")
-		(at 196.615 100.975)
+		(at 196.615 101.475)
 		(descr "Through hole straight pin header, 1x01, 1.00mm pitch, single row")
 		(tags "Through hole pin header THT 1x01 1.00mm single row")
@@
 	(gr_rect
 		(start 179.75 88.25)
-		(end 197.75 101.8)
+		(end 197.75 102.25)
 		(stroke
 			(width 0.05)
@@
 		)
 	)
+	(dimension
+		(type orthogonal)
+		(layer "F.SilkS")
+		(pts
+			(xy 179.75 88.25) (xy 197.75 88.55)
+		)
+		(height -3.75)
+		(orientation 0)
+		(format
+			(prefix "")
+			(suffix "")
+			(units 3)
+			(units_format 0)
+			(precision 4)
+			(suppress_zeroes yes)
+		)
+		(style
+			(thickness 0.1)
+			(arrow_length 1.27)
+			(text_position_mode 0)
+			(arrow_direction outward)
+			(extension_height 0.58642)
+			(extension_offset 0.5)
+			(keep_text_aligned yes)
+		)
+		(gr_text "18"
+			(at 188.75 83.4 0)
+			(layer "F.SilkS")
+			(effects
+				(font
+					(size 1 1)
+					(thickness 0.1)
+				)
+			)
+		)
+	)
+	(dimension
+		(type orthogonal)
+		(layer "F.SilkS")
+		(pts
+			(xy 200 102.25) (xy 198.75 88.25)
+		)
+		(height 0)
+		(orientation 1)
+		(format
+			(prefix "")
+			(suffix "")
+			(units 3)
+			(units_format 0)
+			(precision 4)
+			(suppress_zeroes yes)
+		)
+		(style
+			(thickness 0.1)
+			(arrow_length 1.27)
+			(text_position_mode 2)
+			(arrow_direction outward)
+			(extension_height 0.58642)
+			(extension_offset 0.5)
+			(keep_text_aligned yes)
+		)
+		(gr_text "14"
+			(at 201.5 95.25 90)
+			(layer "F.SilkS")
+			(effects
+				(font
+					(size 1 1)
+					(thickness 0.1)
+				)
+			)
+		)
+	)
 	(segment
 		(start 185.874998 95.125002)
@@
 	(segment
 		(start 180.865 99.535)
-		(end 180.865 101)
+		(end 180.865 101.45)
 		(width 0.6)
 		(layer "F.Cu")
@@
 	)
 	(segment
+		(start 195.9375 96.1875)
+		(end 196.615 96.865)
+		(width 0.6)
+		(layer "F.Cu")
+		(net "+12V")
+	)
+	(segment
 		(start 196.615 96.865)
-		(end 196.615 100.975)
+		(end 196.615 101.45)
+		(width 0.6)
+		(layer "F.Cu")
+		(net "+12V")
+	)
+	(segment
+		(start 192.694998 96.1875)
+		(end 195.9375 96.1875)
 		(width 0.6)
 		(layer "F.Cu")
@@
 		(end 192.694998 96.1875)
 		(width 0.3)
-		(layer "F.Cu")
-		(net "+12V")
-	)
-	(segment
-		(start 195.9375 96.1875)
-		(end 196.615 96.865)
-		(width 0.6)
-		(layer "F.Cu")
-		(net "+12V")
-	)
-	(segment
-		(start 192.694998 96.1875)
-		(end 195.9375 96.1875)
-		(width 0.6)
 		(layer "F.Cu")
 		(net "+12V")
@@
 		(polygon
 			(pts
-				(xy 179.75 88) (xy 198.25 88) (xy 198.25 102) (xy 179.75 102)
-			)
-		)
+				(xy 179.75 88) (xy 198.25 88) (xy 198.25 102.75) (xy 179.75 102.75)
+			)
+		)
